File: PCB-Model/NumpadPCB-V1.1/NumpadPCB-V11.kicad_pcb (KiCad board)
At the start: 2 copper layers, 78.2 x 130.5 mm, 121 parts, among them J1 USB_C_Receptacle, K1 KEYSW, K10 KEYSW, K11 KEYSW, K12 KEYSW, K12B1 KEYSW, K13 KEYSW, K14 KEYSW, K15 KEYSW, K16 KEYSW, K17 KEYSW, K17B1 KEYSW, K18 KEYSW, K19 KEYSW, K2 KEYSW, K20 KEYSW, K20B1 KEYSW, K3 KEYSW, K4 KEYSW, K5 KEYSW, K6 KEYSW, K7 KEYSW, K8 KEYSW, K9 KEYSW, SW1 SW_PUSH, SW2 Rotary_Encoder_Switch, U1 ATMEGA32U4, U2 AO3400, X1 XTAL_GND

Commit message: Add files via upload
Parts:
- removed the C3 at (168.0, 113.4)
- added C8: 0.1u, Capacitor_SMD:C_0805_2012Metric_Pad1.15x1.40mm_HandSolder, B.Cu at (70.2, 72.2)
- L1, L10, L12, L14, L17, L19, L2, L3, L4, L5, L8, L9: moved to F.Cu
- L16B1: renamed from L20B1; moved to F.Cu
- L31: footprint Connector_Wire:SolderWirePad_1x04_P3.81mm_Drill1.2mm -> Connector_PinSocket_2.54mm:PinSocket_1x04_P2.54mm_Vertical; moved to F.Cu
- moved R26 199.8 mm to (45.4, 181.6), turned to 270 degrees
- moved R22 197.5 mm to (45.4, 162.5), turned to 270 degrees
- moved U2 195.2 mm to (47.2, 90.9)
- moved R18 193.7 mm to (45.4, 143.5), turned to 270 degrees
- moved SW1 180.4 mm to (56.1, 74.6), turned to 270 degrees
- moved R1 179.7 mm to (61.6, 72.2), turned to 90 degrees
- moved L17 178.9 mm to (50.5, 182.6)
- moved L9 170.9 mm to (50.5, 144.5)
- moved R10 167.5 mm to (45.4, 105.4), turned to 270 degrees
- moved R15 162.4 mm to (64.5, 124.4), turned to 270 degrees
- moved C1 161.9 mm to (73.8, 72.2), turned to 90 degrees
- moved L10 160.6 mm to (69.5, 144.5)
- moved R6 158.8 mm to (67.9, 82.8), turned to 180 degrees
- moved C7 158.5 mm to (67.9, 79.3), turned to 180 degrees
- moved C5 155.5 mm to (74.8, 93.5), turned to 270 degrees
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- renumbered C4 to C3, C6 to C4, C7 to C5, C5 to C6, C8 to C7, L12B1 to L8B1
Connections:
- J1 pad A4: Net-(J1-PadA4) -> VCC
- J1 pad A9: Net-(J1-PadA4) -> VCC
- J1 pad B4: Net-(J1-PadA4) -> VCC
- J1 pad B9: Net-(J1-PadA4) -> VCC
- K12B1 pad 1: col3 -> Net-(D12-Pad2)
- K12B1 pad 2: Net-(D12-Pad2) -> col3
- K20B1 pad 1: col3 -> Net-(D20-Pad2)
- K20B1 pad 2: Net-(D20-Pad2) -> col3
- L16B1 pad 1: Net-(L20-Pad1) -> Net-(L16-Pad1)
- L8B1 pad 1: Net-(L12-Pad1) -> Net-(L8-Pad1)
- U1 pad 12: BKL -> RGB
- U1 pad 25: Net-(U1-Pad25) -> enB
- U1 pad 26: col3 -> enA
- U1 pad 27: col2 -> row4
- U1 pad 28: col1 -> row3
- U1 pad 29: col0 -> row2
- U1 pad 30: enB -> row1
- U1 pad 31: enA -> row0
- U1 pad 32: RGB -> BKL
- U1 pad 37: row0 -> col3
- U1 pad 38: row1 -> col2
- U1 pad 39: row2 -> col1
- U1 pad 40: row3 -> col0
- U1 pad 41: row4 -> Net-(U1-Pad41)
- U1 pad 7: Net-(J1-PadA4) -> VCC
Routing:
- net VCC: track 0.00 -> 760.2 mm, vias 0 -> 17
- net Net-(R10-Pad1): track 0.00 -> 396.1 mm
- net row4: track 0.00 -> 192.5 mm
- net row3: track 0.00 -> 174.3 mm
- net row2: track 0.00 -> 152.3 mm
- net col0: track 0.00 -> 133.8 mm, vias 0 -> 1
- net row1: track 0.00 -> 132.0 mm
- net col3: track 0.00 -> 128.5 mm, vias 0 -> 1
- net row0: track 0.00 -> 111.8 mm
- net col2: track 0.00 -> 109.4 mm, vias 0 -> 1
- net col1: track 0.00 -> 103.4 mm, vias 0 -> 1
- net Net-(J1-PadA7): track 0.00 -> 45.9 mm, vias 0 -> 2
- net Net-(J1-PadA6): track 0.00 -> 44.7 mm, vias 0 -> 2
- net enSw: track 0.00 -> 39.8 mm, vias 0 -> 1
- net Net-(L25-Pad2): track 0.00 -> 39.2 mm
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- added copper zone on B.Cu, net GND
- added copper zone on F.Cu, net GND
Other:
- outline, holes or cut-outs redrawn
- board text added: "Glowpad V1.1 Carter Cocke"
