File: PCB-Model/NumpadPCB-V1.1/NumpadPCB-V11.sch (KiCad schematic (older format))
At the start: 121 parts, among them J1 USB_C_Receptacle, K1 KEYSW, K10 KEYSW, K11 KEYSW, K12 KEYSW, K12B1 KEYSW, K13 KEYSW, K14 KEYSW, K15 KEYSW, K16 KEYSW, K17 KEYSW, K17B1 KEYSW, K18 KEYSW, K19 KEYSW, K2 KEYSW, K20 KEYSW, K20B1 KEYSW, K3 KEYSW, K4 KEYSW, K5 KEYSW, K6 KEYSW, K7 KEYSW, K8 KEYSW, K9 KEYSW, SW1 SW_PUSH, SW2 Rotary_Encoder_Switch, U1 ATMEGA32U4, U2 AO3400, X1 XTAL_GND

Commit message: Add files via upload
Parts:
- renumbered C4 to C3, C6 to C4, C7 to C5, C5 to C6, C8 to C7, C3 to C8, L20B1 to L16B1, L12B1 to L8B1
Connections:
- net BKL: now also U1.32 (PC7); no longer U1.12 (PB7/~RTS)
- net RGB: now also U1.12 (PB7/~RTS); no longer U1.32 (PC7)
- net VCC: now also J1.A4 (VBUS), J1.A9 (VBUS), J1.B4 (VBUS), J1.B9 (VBUS), U1.7 (VBus)
- net col0: now also U1.40 (PF1); no longer U1.29 (PB5)
- net col1: now also U1.39 (PF4); no longer U1.28 (PB4)
- net col2: now also U1.38 (PF5); no longer U1.27 (T0/PD7)
- net col3: now also K12B1.2, K20B1.2, U1.37 (PF6); no longer K12B1.1, K20B1.1, U1.26 (T1/PD6)
- net enA: now also U1.26 (T1/PD6); no longer U1.31 (PC6)
- net enB: now also U1.25 (ICP1/PD4); no longer U1.30 (PB6)
- net row0: now also U1.31 (PC6); no longer U1.37 (PF6)
- net row1: now also U1.30 (PB6); no longer U1.38 (PF5)
- net row2: now also U1.29 (PB5); no longer U1.39 (PF4)
- net row3: now also U1.28 (PB4); no longer U1.40 (PF1)
- net row4: now also U1.27 (T0/PD7); no longer U1.41 (PF0)
- net at D12.2, K12.2: now also K12B1.1; no longer K12B1.2
- net at D20.2, K20.2: now also K20B1.1; no longer K20B1.2
- net at L8.1 (K), R17.2: now also L8B1.1 (K)
- net at L12.1 (K), R21.2: no longer L8B1.1 (K)
- net at L16.1 (K), R25.2: now also L16B1.1 (K)
- net at L20.1 (K), R29.2: no longer L16B1.1 (K)
Other:
- moved on the sheet: K12B1, K20B1, L10, L11, L12, L16B1, L17, L17B1, L18, L19, L20, L8B1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
