File: keyboards/eyeohdesigns/theboulevard/PCBFiles/blvdtop/blvdtop.kicad_pcb (KiCad board)
At the start: 2 copper layers, 257.2 x 21.4 mm, 13 parts, among them J1 Conn_01x12_Male, K53 KEYSW, K54 KEYSW, K55 KEYSW, K56 KEYSW, SW1 Rotary_Encoder_Switch

Commit message: updated kicad files for theboulevard top PCB
Parts:
- added REF**: MountingHole_2.2mm_M2_Pad, MountingHole:MountingHole_2.2mm_M2_Pad, F.Cu at (118.4, 22.5)
- added REF**: MountingHole_2.2mm_M2_Pad, MountingHole:MountingHole_2.2mm_M2_Pad, F.Cu at (213.6, 22.5)
- D53, D54, D55, D56, D57: value DIODE -> D
- turned D53 to 0 degrees
- turned D54 to 0 degrees
- turned D55 to 0 degrees
- turned D56 to 0 degrees
- turned D57 to 180 degrees
Connections:
- D53 pad 1: Net-(D53-Pad1) -> /Row0
- D53 pad 2: /Row0 -> Net-(D53-Pad2)
- D54 pad 1: Net-(D54-Pad1) -> /Row0
- D54 pad 2: /Row0 -> Net-(D54-Pad2)
- D55 pad 1: Net-(D55-Pad1) -> /Row0
- D55 pad 2: /Row0 -> Net-(D55-Pad2)
- D56 pad 1: Net-(D56-Pad1) -> /Row0
- D56 pad 2: /Row0 -> Net-(D56-Pad2)
- D57 pad 1: Net-(D57-Pad1) -> /Row0
- D57 pad 2: /Row0 -> Net-(D57-Pad2)
- J1 pad 1: /Col10 -> /EncB
- J1 pad 10: /Col1 -> +5V
- J1 pad 11: VCC -> /Col0
- J1 pad 12: /Col0 -> VCC
- J1 pad 2: /EncB -> /Col10
- J1 pad 3: /Col11 -> /EncA
- J1 pad 4: /EncA -> /Col11
- J1 pad 5: /Col12 -> /LEDs
- J1 pad 6: /LEDs -> /Col12
- J1 pad 7: Net-(J1-Pad7) -> /Row0
- J1 pad 8: /Row0 -> Net-(J1-Pad8)
- J1 pad 9: +5V -> /Col1
- K53 pad 2: Net-(D53-Pad1) -> Net-(D53-Pad2)
- K54 pad 2: Net-(D54-Pad1) -> Net-(D54-Pad2)
- K55 pad 2: Net-(D55-Pad1) -> Net-(D55-Pad2)
- K56 pad 2: Net-(D56-Pad1) -> Net-(D56-Pad2)
- SW1 pad S2: Net-(D57-Pad1) -> Net-(D57-Pad2)
Routing:
- net Net-(D57-Pad2): track 0.00 -> 19.0 mm
- net Net-(D57-Pad1): track 19.0 -> 0.00 mm
- net /EncA: track 169.3 -> 157.3 mm, vias 0 -> 1
- net Net-(D56-Pad2): track 0.00 -> 10.5 mm
- net Net-(D56-Pad1): track 10.5 -> 0.00 mm
- net Net-(D55-Pad2): track 0.00 -> 10.5 mm
- net Net-(D55-Pad1): track 10.5 -> 0.00 mm
- net Net-(D54-Pad2): track 0.00 -> 10.5 mm
- net Net-(D54-Pad1): track 10.5 -> 0.00 mm
- net Net-(D53-Pad2): track 0.00 -> 10.5 mm
- net Net-(D53-Pad1): track 10.5 -> 0.00 mm
- net /Row0: track 274.5 -> 264.5 mm, vias 1 -> 0
- net /EncB: track 156.9 -> 150.6 mm
- net /Col12: track 103.3 -> 98.0 mm
- net /Col11: track 87.3 -> 82.4 mm, vias 2 -> 1
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Other:
- board text added: "Blvd Top Ver P2"
