File: keyboards/eyeohdesigns/theboulevard/PCBFiles/blvdtop/blvdtop.sch (KiCad schematic (older format))
At the start: 13 parts, among them J1 Conn_01x12_Male, K53 KEYSW, K54 KEYSW, K55 KEYSW, K56 KEYSW, SW1 Rotary_Encoder_Switch

Commit message: updated kicad files for theboulevard top PCB
Parts:
- removed D53, D54, D55, D56, D57: DIODE, keyboard_parts:D_SOD123, symbol pspice:DIODE
- added D53, D54, D55, D56, D57: D, keyboard_parts:D_SOD123, symbol Device:D
- LED1, LED2: symbol keybage:WS2812B -> blvdtop-rescue:WS2812B-keybage
Connections:
- wire segments 19 -> 24
Other:
- moved on the sheet: J1
Changed lines of the file:
@@
 L Connector:Conn_01x12_Male J1
 U 1 1 6193240B
-P 9800 2050
-F 0 "J1" H 9908 2731 50  0000 C CNN
-F 1 "Conn_01x12_Male" H 9908 2640 50  0000 C CNN
-F 2 "Connector_PinHeader_2.00mm:PinHeader_2x06_P2.00mm_Vertical" H 9800 2050 50  0001 C CNN
-F 3 "~" H 9800 2050 50  0001 C CNN
-	1    9800 2050
+P 9700 2050
+F 0 "J1" H 9808 2731 50  0000 C CNN
+F 1 "Conn_01x12_Male" H 9808 2640 50  0000 C CNN
+F 2 "Connector_PinHeader_2.00mm:PinHeader_2x06_P2.00mm_Vertical" H 9700 2050 50  0001 C CNN
+F 3 "~" H 9700 2050 50  0001 C CNN
+	1    9700 2050
 	1    0    0    -1
 $EndComp
@@
 $EndComp
 $Comp
-L keybage:WS2812B LED1
+L blvdtop-rescue:WS2812B-keybage LED1
 U 1 1 61937713
 P 3150 1150
@@
 $EndComp
 $Comp
-L keybage:WS2812B LED2
+L blvdtop-rescue:WS2812B-keybage LED2
 U 1 1 619382FF
 P 4900 1150
@@
 	1    0    0    -1
 $EndComp
-$Comp
-L pspice:DIODE D53
-U 1 1 6193C8DD
-P 2950 3950
-F 0 "D53" V 2904 4078 50  0000 L CNN
-F 1 "DIODE" V 2995 4078 50  0000 L CNN
-F 2 "keyboard_parts:D_SOD123" H 2950 3950 50  0001 C CNN
-F 3 "~" H 2950 3950 50  0001 C CNN
-	1    2950 3950
-	0    1    1    0
-$EndComp
-$Comp
-L pspice:DIODE D54
-U 1 1 6193D64B
-P 3700 3950
-F 0 "D54" V 3654 4078 50  0000 L CNN
-F 1 "DIODE" V 3745 4078 50  0000 L CNN
-F 2 "keyboard_parts:D_SOD123" H 3700 3950 50  0001 C CNN
-F 3 "~" H 3700 3950 50  0001 C CNN
-	1    3700 3950
-	0    1    1    0
-$EndComp
-$Comp
-L pspice:DIODE D55
-U 1 1 6193D8FC
-P 4650 3950
-F 0 "D55" V 4604 4078 50  0000 L CNN
-F 1 "DIODE" V 4695 4078 50  0000 L CNN
-F 2 "keyboard_parts:D_SOD123" H 4650 3950 50  0001 C CNN
-F 3 "~" H 4650 3950 50  0001 C CNN
-	1    4650 3950
-	0    1    1    0
-$EndComp
-$Comp
-L pspice:DIODE D56
-U 1 1 6193DA25
-P 5400 3950
-F 0 "D56" V 5354 4078 50  0000 L CNN
-F 1 "DIODE" V 5445 4078 50  0000 L CNN
-F 2 "keyboard_parts:D_SOD123" H 5400 3950 50  0001 C CNN
-F 3 "~" H 5400 3950 50  0001 C CNN
-	1    5400 3950
-	0    1    1    0
-$EndComp
-$Comp
-L pspice:DIODE D57
-U 1 1 6193DD63
-P 2100 3950
-F 0 "D57" V 2054 4078 50  0000 L CNN
-F 1 "DIODE" V 2145 4078 50  0000 L CNN
-F 2 "keyboard_parts:D_SOD123" H 2100 3950 50  0001 C CNN
-F 3 "~" H 2100 3950 50  0001 C CNN
-	1    2100 3950
-	0    1    1    0
-$EndComp
 Wire Wire Line
 	2650 1350 2650 1850
@@
 Wire Wire Line
 	5700 950  5400 950
-Text Label 10000 2050 0    50   ~ 0
+Text Label 9900 1950 0    50   ~ 0
 LEDs
-Text Label 10000 1850 0    50   ~ 0
+Text Label 9900 1750 0    50   ~ 0
 EncA
-Text Label 10000 1650 0    50   ~ 0
+Text Label 9900 1550 0    50   ~ 0
 EncB
 Text Label 5950 4150 0    50   ~ 0
 Row0
-Text Label 10000 2650 0    50   ~ 0
+Text Label 9900 2550 0    50   ~ 0
 Col0
-Text Label 10000 1950 0    50   ~ 0
+Text Label 9900 2050 0    50   ~ 0
 Col12
-Text Label 10000 1750 0    50   ~ 0
+Text Label 9900 1850 0    50   ~ 0
 Col11
-Text Label 10000 1550 0    50   ~ 0
+Text Label 9900 1650 0    50   ~ 0
 Col10
-Text Label 10000 2450 0    50   ~ 0
+Text Label 9900 2350 0    50   ~ 0
 Col1
 $Comp
 L power:VCC #PWR0101
 U 1 1 61940884
-P 10000 2550
-F 0 "#PWR0101" H 10000 2400 50  0001 C CNN
-F 1 "VCC" H 10017 2723 50  0000 C CNN
-F 2 "" H 10000 2550 50  0001 C CNN
-F 3 "" H 10000 2550 50  0001 C CNN
-	1    10000 2550
+P 9900 2650
+F 0 "#PWR0101" H 9900 2500 50  0001 C CNN
+F 1 "VCC" H 9917 2823 50  0000 C CNN
+F 2 "" H 9900 2650 50  0001 C CNN
+F 3 "" H 9900 2650 50  0001 C CNN
+	1    9900 2650
 	0    1    1    0
 $EndComp
@@
 	5400 3450 5400 3750
 Wire Wire Line
-	2100 4150 2950 4150
-Connection ~ 2950 4150
-Wire Wire Line
-	2950 4150 3700 4150
-Connection ~ 3700 4150
-Wire Wire Line
-	3700 4150 4650 4150
-Connection ~ 4650 4150
-Wire Wire Line
-	4650 4150 5400 4150
-Wire Wire Line
-	5950 4150 5400 4150
-Connection ~ 5400 4150
-Wire Wire Line
 	2100 3450 2100 3750
-Text Label 10000 2250 0    50   ~ 0
+Text Label 9900 2150 0    50   ~ 0
 Row0
 $Comp
 L keyboard_parts:GND #PWR0107
 U 1 1 619BA511
-P 10000 2350
-F 0 "#PWR0107" H 10000 2400 20  0001 C CNN
-F 1 "GND" H 10000 2250 30  0000 C CNN
-F 2 "" H 10000 2350 60  0000 C CNN
-F 3 "" H 10000 2350 60  0000 C CNN
-	1    10000 2350
+P 9900 2450
+F 0 "#PWR0107" H 9900 2500 20  0001 C CNN
+F 1 "GND" H 9900 2350 30  0000 C CNN
+F 2 "" H 9900 2450 60  0000 C CNN
+F 3 "" H 9900 2450 60  0000 C CNN
+	1    9900 2450
 	0    -1   -1   0
 $EndComp
 Wire Wire Line
 	2200 2500 2200 2850
+$Comp
+L Device:D D56
+U 1 1 605797E2
+P 5400 3900
+F 0 "D56" V 5446 3821 50  0000 R CNN
+F 1 "D" V 5355 3821 50  0000 R CNN
+F 2 "keyboard_parts:D_SOD123" H 5400 3900 50  0001 C CNN
+F 3 "~" H 5400 3900 50  0001 C CNN
+	1    5400 3900
+	0    -1   -1   0
+$EndComp
+$Comp
+L Device:D D55
+U 1 1 6057A422
+P 4650 3900
+F 0 "D55" V 4696 3821 50  0000 R CNN
+F 1 "D" V 4605 3821 50  0000 R CNN
+F 2 "keyboard_parts:D_SOD123" H 4650 3900 50  0001 C CNN
+F 3 "~" H 4650 3900 50  0001 C CNN
+	1    4650 3900
+	0    -1   -1   0
+$EndComp
+$Comp
+L Device:D D54
+U 1 1 6057A7D6
+P 3700 3900
+F 0 "D54" V 3746 3821 50  0000 R CNN
+F 1 "D" V 3655 3821 50  0000 R CNN
+F 2 "keyboard_parts:D_SOD123" H 3700 3900 50  0001 C CNN
+F 3 "~" H 3700 3900 50  0001 C CNN
+	1    3700 3900
+	0    -1   -1   0
+$EndComp
+$Comp
+L Device:D D53
+U 1 1 6057A7DC
+P 2950 3900
+F 0 "D53" V 2996 3821 50  0000 R CNN
+F 1 "D" V 2905 3821 50  0000 R CNN
+F 2 "keyboard_parts:D_SOD123" H 2950 3900 50  0001 C CNN
+F 3 "~" H 2950 3900 50  0001 C CNN
+	1    2950 3900
+	0    -1   -1   0
+$EndComp
+$Comp
+L Device:D D57
+U 1 1 6057AB76
+P 2100 3900
+F 0 "D57" V 2146 3821 50  0000 R CNN
+F 1 "D" V 2055 3821 50  0000 R CNN
+F 2 "keyboard_parts:D_SOD123" H 2100 3900 50  0001 C CNN
+F 3 "~" H 2100 3900 50  0001 C CNN
+	1    2100 3900
+	0    -1   -1   0
+$EndComp
+Wire Wire Line
+	2100 4150 2950 4150
+Wire Wire Line
+	2100 4050 2100 4150
+Wire Wire Line
+	2950 4050 2950 4150
+Connection ~ 2950 4150
+Wire Wire Line
+	2950 4150 3700 4150
+Wire Wire Line
+	3700 4050 3700 4150
+Connection ~ 3700 4150
+Wire Wire Line
+	3700 4150 4650 4150
+Wire Wire Line
+	4650 4050 4650 4150
+Connection ~ 4650 4150
+Wire Wire Line
+	4650 4150 5400 4150
+Wire Wire Line
+	5400 4050 5400 4150
+Connection ~ 5400 4150
+Wire Wire Line
+	5400 4150 5950 4150
 $EndSCHEMATC
